Commit message: simulation complete

File: description/robot.urdf.xacro (robot description, xacro)
@@ -2,3 +2,4 @@
 <robot xmlns:xacro="http://www.ros.org/wiki/xacro"  name="robot">
     <xacro:include filename ="robot_core.xacro" />
+    <xacro:include filename="gazebo_control.xacro"/>
 </robot>

File: description/robot_core.xacro (robot description, xacro)
@@ -264,4 +264,6 @@
         <origin xyz="-0.0055 0.08 0" rpy="-${pi/2} 0 0"/>
         <axis xyz="0 0 1"/>
+        <limit effort="100" velocity="10.0"/>
+        <dynamics damping="0.1" friction="0.1"/>
     </joint>
     <link name="left_wheel">
@@ -287,4 +289,6 @@
         <origin xyz="-0.0055 -0.08 0" rpy="${pi/2} 0 0"/>
         <axis xyz="0 0 -1"/>
+        <limit effort="100" velocity="10.0"/>
+        <dynamics damping="0.1" friction="0.1"/>
     </joint>
     <link name="right_wheel">
