Commit message: working lidar added

File: description/gazebo_control.xacro (robot description, xacro)
@@ -3,45 +3,23 @@
     <!-- Control Parameters -->
     <xacro:property name="max_linear_acceleration" value="10"/>
-    <!-- Gazebo Parameters adding friction by decreasing mu -->
-    <gazebo reference="back_chassis">
-        <mu1>1.0</mu1>
-        <mu2>1.0</mu2>
-    </gazebo>
-    <gazebo reference="right_wheel">
-        <mu1>1.0</mu1>
-        <mu2>1.0</mu2>
-    </gazebo>
-    <gazebo reference="left_wheel">
-        <mu1>1.0</mu1>
-        <mu2>1.0</mu2>
-    </gazebo>
-    <gazebo reference="caster_wheel">
-        <mu1>0.000001</mu1>
-        <mu2>0.000001</mu2>
-    </gazebo>
     <gazebo>
-        <plugin filename="gz-sim-diff-drive-system" name="gz::sim::systems::DiffDrive">
-            <!--Wheel information-->
-            <right_joint>right_wheel_joint</right_joint>
-            <left_joint>left_wheel_joint</left_joint>
-            <wheel_separation>0.212</wheel_separation>
-            <wheel_radius>0.03</wheel_radius>
-            <!-- Limits-->
-            <max_linear_acceleration>${max_linear_acceleration}</max_linear_acceleration>
-            <!-- Output -->
-            <odometry_frame>odom</odometry_frame>
-            <robot_base_frame>base_link</robot_base_frame>
-            <publish_odom>true</publish_odom>
-            <publish_odom_tf>true</publish_odom_tf>
-            <publish_wheel_tf>true</publish_wheel_tf>
-            <odom_publish_frequency>1</odom_publish_frequency>
-            <topic>cmd_vel</topic>
-            <odom_topic>odom</odom_topic>
-        </plugin>
-        <plugin filename="gz-sim-joint-state-publisher-system" name="gz::sim::systems::JointStatePublisher">
-            <topic>joint_states</topic>
-            <joint_name>right_wheel_joint</joint_name>
-            <joint_name>left_wheel_joint</joint_name>
-        </plugin>
-    </gazebo>
+      <plugin filename="gz-sim-diff-drive-system" name="gz::sim::systems::DiffDrive">
+         <right_joint>right_wheel_joint</right_joint>
+         <left_joint>left_wheel_joint</left_joint>
+         <wheel_separation>0.212</wheel_separation>
+         <wheel_diameter>0.03</wheel_diameter>
+         <max_linear_acceleration>40</max_linear_acceleration>
+         <topic>cmd_vel</topic>
+         <odom_topic>odom</odom_topic>
+         <frame_id>odom</frame_id>
+         <child_frame_id>base_link</child_frame_id>
+         <odom_publisher_frequency>100</odom_publisher_frequency>
+         <tf_topic>/tf</tf_topic>
+      </plugin>
+      <plugin filename="gz-sim-joint-state-publisher-system" name="gz::sim::systems::JointStatePublisher">
+         <topic>joint_states</topic>
+         <joint_name>right_wheel_joint</joint_name>
+         <joint_name>left_wheel_joint</joint_name>
+      </plugin>
+   </gazebo>
 </robot>

File: description/robot.urdf.xacro (robot description, xacro)
@@ -3,3 +3,4 @@
     <xacro:include filename ="robot_core_v2.xacro" />
     <xacro:include filename="gazebo_control.xacro"/>
+    <xacro:include filename="lidar.xacro"/>
 </robot>

File: description/robot_core_v2.xacro (robot description, xacro)
@@ -14,12 +14,15 @@
         <color rgba="0 0 0 1" />
     </material>
+    <material name ="red">
+        <color rgba="1 0 0 1" />
+    </material>
     <link name="base_link">
     </link>
     <joint name="chassis_joint" type="fixed">
         <parent link= "base_link"/>
-        <child link="midle_chassis"/>
+        <child link="chassis"/>
         <origin xyz="-0.069 0 0"/>
     </joint>
-    <link name="midle_chassis">
+    <link name="chassis">
         <visual>
             <origin xyz="0 0 0.0025"/>
@@ -74,80 +77,80 @@
         <!-- Front_Right_spacer -->
         <visual>
-            <origin xyz="0.115 0.0875 0.0225"/>
-            <geometry>
-                <cylinder radius = "0.0055" length="0.04"/>
-            </geometry>
-            <material name="white"/>
-        </visual>
-        <collision>
-            <origin xyz="0.115 0.0875 0.0225"/>
-            <geometry>
-                <cylinder radius = "0.0055" length="0.04"/>
-            </geometry>
-        </collision>
-        <xacro:inertial_cylinder mass="0.005" length="0.04" radius="0.0055">
-            <origin xyz= "0.115 0.0875 0.0225" rpy="0 0 0"/>
+            <origin xyz="0.115 0.0875 0.025"/>
+            <geometry>
+                <cylinder radius = "0.0055" length="0.045"/>
+            </geometry>
+            <material name="white"/>
+        </visual>
+        <collision>
+            <origin xyz="0.115 0.0875 0.025"/>
+            <geometry>
+                <cylinder radius = "0.0055" length="0.045"/>
+            </geometry>
+        </collision>
+        <xacro:inertial_cylinder mass="0.005" length="0.04" radius="0.0055">
+            <origin xyz= "0.115 0.0875 0.025" rpy="0 0 0"/>
         </xacro:inertial_cylinder>
         <!-- Front_Left_spacer -->
         <visual>
-            <origin xyz="0.115 -0.0875 0.0225"/>
-            <geometry>
-                <cylinder radius = "0.0055" length="0.04"/>
-            </geometry>
-            <material name="white"/>
-        </visual>
-        <collision>
-            <origin xyz="0.115 -0.0875 0.0225"/>
-            <geometry>
-                <cylinder radius = "0.0055" length="0.04"/>
-            </geometry>
-        </collision>
-        <xacro:inertial_cylinder mass="0.005" length="0.04" radius="0.0055">
-            <origin xyz= "0.115 -0.0875 0.0225" rpy="0 0 0"/>
+            <origin xyz="0.115 -0.0875 0.025"/>
+            <geometry>
+                <cylinder radius = "0.0055" length="0.045"/>
+            </geometry>
+            <material name="white"/>
+        </visual>
+        <collision>
+            <origin xyz="0.115 -0.0875 0.025"/>
+            <geometry>
+                <cylinder radius = "0.0055" length="0.045"/>
+            </geometry>
+        </collision>
+        <xacro:inertial_cylinder mass="0.005" length="0.04" radius="0.0055">
+            <origin xyz= "0.115 -0.0875 0.025" rpy="0 0 0"/>
         </xacro:inertial_cylinder>
         <!-- Back_Right_spacer -->
         <visual>
-            <origin xyz="-0.115 0.0875 0.0225"/>
-            <geometry>
-                <cylinder radius = "0.0055" length="0.04"/>
-            </geometry>
-            <material name="white"/>
-        </visual>
-        <collision>
-            <origin xyz="-0.115 0.0875 0.0225"/>
-            <geometry>
-                <cylinder radius = "0.0055" length="0.04"/>
-            </geometry>
-        </collision>
-        <xacro:inertial_cylinder mass="0.005" length="0.04" radius="0.0055">
-            <origin xyz= "-0.115 0.0875 0.0225" rpy="0 0 0"/>
+            <origin xyz="-0.115 0.0875 0.025"/>
+            <geometry>
+                <cylinder radius = "0.0055" length="0.045"/>
+            </geometry>
+            <material name="white"/>
+        </visual>
+        <collision>
+            <origin xyz="-0.115 0.0875 0.025"/>
+            <geometry>
+                <cylinder radius = "0.0055" length="0.045"/>
+            </geometry>
+        </collision>
+        <xacro:inertial_cylinder mass="0.005" length="0.04" radius="0.0055">
+            <origin xyz= "-0.115 0.0875 0.025" rpy="0 0 0"/>
         </xacro:inertial_cylinder>
         <!-- Back_left_spacer -->
         <visual>
-            <origin xyz="-0.115 -0.0875 0.0225"/>
-            <geometry>
-                <cylinder radius = "0.0055" length="0.04"/>
-            </geometry>
-            <material name="white"/>
-        </visual>
-        <collision>
-            <origin xyz="-0.115 -0.0875 0.0225"/>
-            <geometry>
-                <cylinder radius = "0.0055" length="0.04"/>
-            </geometry>
-        </collision>
-        <xacro:inertial_cylinder mass="0.005" length="0.04" radius="0.0055">
-            <origin xyz= "-0.115 -0.0875 0.0225" rpy="0 0 0"/>
+            <origin xyz="-0.115 -0.0875 0.025"/>
+            <geometry>
+                <cylinder radius = "0.0055" length="0.045"/>
+            </geometry>
+            <material name="white"/>
+        </visual>
+        <collision>
+            <origin xyz="-0.115 -0.0875 0.025"/>
+            <geometry>
+                <cylinder radius = "0.0055" length="0.045"/>
+            </geometry>
+        </collision>
+        <xacro:inertial_cylinder mass="0.005" length="0.04" radius="0.0055">
+            <origin xyz= "-0.115 -0.0875 0.025" rpy="0 0 0"/>
         </xacro:inertial_cylinder>
         <!--Second stage-->                                     <!--Second stage-->
         <visual>
-            <origin xyz="0 0 0.0425"/>
-            <geometry>
-                <box size="0.2 0.15 0.005"/>
-            </geometry>
-            <material name="white"/>
-        </visual>
-        <collision>
-            <origin xyz="0 0 0.0425"/>
+            <origin xyz="0 0 0.045"/>
+            <geometry>
+                <box size="0.2 0.15 0.005"/>
+            </geometry>
+            <material name="white"/>
+        </visual>
+        <collision>
+            <origin xyz="0 0 0.045"/>
             <geometry>
                 <box size="0.2 0.15 0.005"/>
@@ -155,118 +158,118 @@
         </collision>
         <xacro:inertial_box mass="0.015" x="0.2" y="0.15" z="0.005">
-            <origin xyz= "0 0 0.0425" rpy="0 0 0"/>
+            <origin xyz= "0 0 0.045" rpy="0 0 0"/>
         </xacro:inertial_box>
         <!-- front chassis -->
         <visual>
-            <origin xyz="0.115 0 0.0425"/>
-            <geometry>
-                <box size="0.03 0.2 0.005"/>
-            </geometry>
-            <material name="white"/>
-        </visual>
-        <collision>
-            <origin xyz="0.115 0 0.0425"/>
-            <geometry>
-                <box size="0.03 0.2 0.005"/>
-            </geometry>
-        </collision>
-        <xacro:inertial_box mass="0.005" x="0.03" y="0.2" z="0.005">
-            <origin xyz= "0.115 0 0.0425" rpy="0 0 0"/>
+            <origin xyz="0.115 0 0.045"/>
+            <geometry>
+                <box size="0.03 0.2 0.005"/>
+            </geometry>
+            <material name="white"/>
+        </visual>
+        <collision>
+            <origin xyz="0.115 0 0.045"/>
+            <geometry>
+                <box size="0.03 0.2 0.005"/>
+            </geometry>
+        </collision>
+        <xacro:inertial_box mass="0.005" x="0.03" y="0.2" z="0.005">
+            <origin xyz= "0.115 0 0.045" rpy="0 0 0"/>
         </xacro:inertial_box>
         <!-- back chassis -->
         <visual>
-            <origin xyz="-0.115 0 0.0425"/>
-            <geometry>
-                <box size="0.03 0.2 0.005"/>
-            </geometry>
-            <material name="white"/>
-        </visual>
-        <collision>
-            <origin xyz="-0.115 0 0.0425"/>
-            <geometry>
-                <box size="0.03 0.2 0.005"/>
-            </geometry>
-        </collision>
-        <xacro:inertial_box mass="0.005" x="0.03" y="0.2" z="0.005">
-            <origin xyz= "-0.115 0 0.0425" rpy="0 0 0"/>
+            <origin xyz="-0.115 0 0.045"/>
+            <geometry>
+                <box size="0.03 0.2 0.005"/>
+            </geometry>
+            <material name="white"/>
+        </visual>
+        <collision>
+            <origin xyz="-0.115 0 0.045"/>
+            <geometry>
+                <box size="0.03 0.2 0.005"/>
+            </geometry>
+        </collision>
+        <xacro:inertial_box mass="0.005" x="0.03" y="0.2" z="0.005">
+            <origin xyz= "-0.115 0 0.045" rpy="0 0 0"/>
         </xacro:inertial_box>
         <!-- Front_Right_spacer -->
         <visual>
-            <origin xyz="0.115 0.0875 0.0625"/>
-            <geometry>
-                <cylinder radius = "0.0055" length="0.04"/>
-            </geometry>
-            <material name="white"/>
-        </visual>
-        <collision>
-            <origin xyz="0.115 0.0875 0.0625"/>
-            <geometry>
-                <cylinder radius = "0.0055" length="0.04"/>
-            </geometry>
-        </collision>
-        <xacro:inertial_cylinder mass="0.005" length="0.04" radius="0.0055">
-            <origin xyz= "0.115 0.0875 0.0625" rpy="0 0 0"/>
+            <origin xyz="0.115 0.0875 0.065"/>
+            <geometry>
+                <cylinder radius = "0.0055" length="0.045"/>
+            </geometry>
+            <material name="white"/>
+        </visual>
+        <collision>
+            <origin xyz="0.115 0.0875 0.065"/>
+            <geometry>
+                <cylinder radius = "0.0055" length="0.045"/>
+            </geometry>
+        </collision>
+        <xacro:inertial_cylinder mass="0.005" length="0.04" radius="0.0055">
+            <origin xyz= "0.115 0.0875 0.065" rpy="0 0 0"/>
         </xacro:inertial_cylinder>
         <!-- Front_Left_spacer -->
         <visual>
-            <origin xyz="0.115 -0.0875 0.0625"/>
-            <geometry>
-                <cylinder radius = "0.0055" length="0.04"/>
-            </geometry>
-            <material name="white"/>
-        </visual>
-        <collision>
-            <origin xyz="0.115 -0.0875 0.0625"/>
-            <geometry>
-                <cylinder radius = "0.0055" length="0.04"/>
-            </geometry>
-        </collision>
-        <xacro:inertial_cylinder mass="0.005" length="0.04" radius="0.0055">
-            <origin xyz= "0.115 -0.0875 0.0625" rpy="0 0 0"/>
+            <origin xyz="0.115 -0.0875 0.065"/>
+            <geometry>
+                <cylinder radius = "0.0055" length="0.045"/>
+            </geometry>
+            <material name="white"/>
+        </visual>
+        <collision>
+            <origin xyz="0.115 -0.0875 0.065"/>
+            <geometry>
+                <cylinder radius = "0.0055" length="0.045"/>
+            </geometry>
+        </collision>
+        <xacro:inertial_cylinder mass="0.005" length="0.04" radius="0.0055">
+            <origin xyz= "0.115 -0.0875 0.065" rpy="0 0 0"/>
         </xacro:inertial_cylinder>
         <!-- Back_Right_spacer -->
         <visual>
-            <origin xyz="-0.115 0.0875 0.0625"/>
-            <geometry>
-                <cylinder radius = "0.0055" length="0.04"/>
-            </geometry>
-            <material name="white"/>
-        </visual>
-        <collision>
-            <origin xyz="-0.115 0.0875 0.0625"/>
-            <geometry>
-                <cylinder radius = "0.0055" length="0.04"/>
-            </geometry>
-        </collision>
-        <xacro:inertial_cylinder mass="0.005" length="0.04" radius="0.0055">
-            <origin xyz= "-0.115 0.0875 0.0625" rpy="0 0 0"/>
+            <origin xyz="-0.115 0.0875 0.065"/>
+            <geometry>
+                <cylinder radius = "0.0055" length="0.045"/>
+            </geometry>
+            <material name="white"/>
+        </visual>
+        <collision>
+            <origin xyz="-0.115 0.0875 0.065"/>
+            <geometry>
+                <cylinder radius = "0.0055" length="0.045"/>
+            </geometry>
+        </collision>
+        <xacro:inertial_cylinder mass="0.005" length="0.04" radius="0.0055">
+            <origin xyz= "-0.115 0.0875 0.065" rpy="0 0 0"/>
         </xacro:inertial_cylinder>
         <!-- Back_left_spacer -->
         <visual>
-            <origin xyz="-0.115 -0.0875 0.0625"/>
-            <geometry>
-                <cylinder radius = "0.0055" length="0.04"/>
-            </geometry>
-            <material name="white"/>
-        </visual>
-        <collision>
-            <origin xyz="-0.115 -0.0875 0.0625"/>
-            <geometry>
-                <cylinder radius = "0.0055" length="0.04"/>
-            </geometry>
-        </collision>
-        <xacro:inertial_cylinder mass="0.005" length="0.04" radius="0.0055">
-            <origin xyz= "-0.115 -0.0875 0.0625" rpy="0 0 0"/>
+            <origin xyz="-0.115 -0.0875 0.065"/>
+            <geometry>
+                <cylinder radius = "0.0055" length="0.045"/>
+            </geometry>
+            <material name="white"/>
+        </visual>
+        <collision>
+            <origin xyz="-0.115 -0.0875 0.065"/>
+            <geometry>
+                <cylinder radius = "0.0055" length="0.045"/>
+            </geometry>
+        </collision>
+        <xacro:inertial_cylinder mass="0.005" length="0.04" radius="0.0055">
+            <origin xyz= "-0.115 -0.0875 0.065" rpy="0 0 0"/>
         </xacro:inertial_cylinder>
         <!--Third stage-->                                     <!--Third stage-->
         <visual>
-            <origin xyz="0 0 0.0825"/>
-            <geometry>
-                <box size="0.2 0.15 0.005"/>
-            </geometry>
-            <material name="white"/>
-        </visual>
-        <collision>
-            <origin xyz="0 0 0.0825"/>
+            <origin xyz="0 0 0.085"/>
+            <geometry>
+                <box size="0.2 0.15 0.005"/>
+            </geometry>
+            <material name="white"/>
+        </visual>
+        <collision>
+            <origin xyz="0 0 0.085"/>
             <geometry>
                 <box size="0.2 0.15 0.005"/>
@@ -274,39 +277,39 @@
         </collision>
         <xacro:inertial_box mass="0.015" x="0.2" y="0.15" z="0.005">
-            <origin xyz= "0 0 0.0825" rpy="0 0 0"/>
+            <origin xyz= "0 0 0.085" rpy="0 0 0"/>
         </xacro:inertial_box>
         <!-- front chassis -->
         <visual>
-            <origin xyz="0.115 0 0.0825"/>
-            <geometry>
-                <box size="0.03 0.2 0.005"/>
-            </geometry>
-            <material name="white"/>
-        </visual>
-        <collision>
-            <origin xyz="0.115 0 0.0825"/>
-            <geometry>
-                <box size="0.03 0.2 0.005"/>
-            </geometry>
-        </collision>
-        <xacro:inertial_box mass="0.005" x="0.03" y="0.2" z="0.005">
-            <origin xyz= "0.115 0 0.0825" rpy="0 0 0"/>
+            <origin xyz="0.115 0 0.085"/>
+            <geometry>
+                <box size="0.03 0.2 0.005"/>
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